Commit message: add lidar link and navigation package

File: src/amr_coco_description/robot/visual/sensor.xacro (robot description, xacro)
@@ -3,5 +3,5 @@
   <!-- Contents-->
   <xacro:macro name="sensor_link" params="">
-    <link name="imu_link"/>
+    <link name="imu_link" />
     <joint name="imu_mount" type="fixed">
       <parent link="base_link" />
@@ -9,4 +9,16 @@
       <origin xyz="0 0 0" rpy="0 0 0" />
     </joint>
+    <link name="laser">
+      <visual>
+        <geometry>
+          <cylinder length="0.04" radius="0.035" />
+        </geometry>
+      </visual>
+    </link>
+    <joint name="lidar_mount" type="fixed">
+      <origin xyz="0.0 0.0 0.20" />
+      <parent link="base_link" />
+      <child link="laser" />
+    </joint>
   </xacro:macro>
 </robot>
